File: CTR-0/CTR-0.kicad_sch (KiCad schematic)
At the start: 1 part, among them U1 RP2040

Commit message: Add files via upload
Parts:
- added C1, C2: 10u, symbol Device:C
- added C3, C4: 15p, symbol Device:C
- added C5: 5u, symbol Device:C
- added J1: USB_C_Receptacle_USB2.0_14P, symbol Connector:USB_C_Receptacle_USB2.0_14P
- added J2, J3: Conn_01x20, symbol Connector_Generic:Conn_01x20
- added J4: Conn_01x03, symbol Connector_Generic:Conn_01x03
- added R1, R2: 5.1K, symbol Device:R
- added R3: 1K, symbol Device:R
- added R4, R5: R, symbol Device:R
- added R6: 10k, symbol Device:R
- added R7: 1k, symbol Device:R
- added SW1: SW_Push, symbol Switch:SW_Push
- added U2: NCP1117-3.3_SOT223, Package_TO_SOT_SMD:SOT-223-3_TabPin2, symbol Regulator_Linear:NCP1117-3.3_SOT223
- added U3: W25Q128JVS, Package_SO:SOIC-8_5.3x5.3mm_P1.27mm, symbol Memory_Flash:W25Q128JVS
- added Y1: Crystal_GND24, symbol Device:Crystal_GND24
Connections:
- net GND: now also U1.19 (TESTEN), C1.2, C2.2, C3.1, C4.1, C5.1, J1.A1 (GND), J1.A12 (GND), J1.B1 (GND), J1.B12 (GND), J1.S1 (SHIELD), R1.2, R2.2, U2.1 (GND), U3.4 (GND), Y1.2, Y1.4
- net +3V3: now reaches U1.1 (IOVDD), U1.10 (IOVDD), U1.22 (IOVDD), U1.33 (IOVDD), U1.42 (IOVDD), U1.49 (IOVDD)
- net +3V3: now also U1.43 (ADC_AVDD), U1.44 (VREG_IN), U1.48 (USB_VDD), C2.1, R6.1, U2.2 (VO), U3.8 (VCC)
- net GPIO8: now reaches U1.11 (GPIO8)
- net GPIO8: now also J2.11 (Pin_11)
- net GPIO9: now reaches U1.12 (GPIO9)
- net GPIO9: now also J2.12 (Pin_12)
- net GPIO10: now reaches U1.13 (GPIO10)
- net GPIO10: now also J2.14 (Pin_14)
- net GPIO11: now reaches U1.14 (GPIO11)
- net GPIO11: now also J2.15 (Pin_15)
- net GPIO12: now reaches U1.15 (GPIO12)
- net GPIO12: now also J2.16 (Pin_16)
- net GPIO13: now reaches U1.16 (GPIO13)
- net GPIO13: now also J2.17 (Pin_17)
- net GPIO14: now reaches U1.17 (GPIO14)
- net GPIO14: now also J2.19 (Pin_19)
- net GPIO15: now reaches U1.18 (GPIO15)
- net GPIO15: now also J2.20 (Pin_20)
- net GPIO0: now reaches U1.2 (GPIO0)
- net GPIO0: now also J2.1 (Pin_1)
- net XIN: now reaches U1.20 (XIN)
- net XIN: now also C3.2, Y1.3
- net XOUT: now reaches U1.21 (XOUT)
- net XOUT: now also R3.2
- net +1V1: now reaches U1.23 (DVDD), U1.50 (DVDD)
- net +1V1: now also U1.45 (VREG_VOUT)
- net SWCLK: now reaches U1.24 (SWCLK)
- net SWD: now reaches U1.25 (SWD)
- net GPIO16: now reaches U1.27 (GPIO16)
- net GPIO17: now reaches U1.28 (GPIO17)
- net GPIO18: now reaches U1.29 (GPIO18)
- net GPIO1: now reaches U1.3 (GPIO1)
- net GPIO1: now also J2.2 (Pin_2)
- net GPIO19: now reaches U1.30 (GPIO19)
- net GPIO20: now reaches U1.31 (GPIO20)
- net GPIO21: now reaches U1.32 (GPIO21)
- net GPIO22: now reaches U1.34 (GPIO22)
- net GPIO23: now reaches U1.35 (GPIO23)
- net GPIO23: now also J3.10 (Pin_10)
- net GPIO24: now reaches U1.36 (GPIO24)
- net GPIO24: now also J3.9 (Pin_9)
- net GPIO25: now reaches U1.37 (GPIO25)
- net GPIO26_ADC0: now reaches U1.38 (GPIO26_ADC0)
- net GPIO26_ADC0: now also J3.5 (Pin_5)
- net GPIO27_ADC1: now reaches U1.39 (GPIO27_ADC1)
- net GPIO2: now reaches U1.4 (GPIO2)
- net GPIO2: now also J2.4 (Pin_4)
- net GPIO28_ADC2: now reaches U1.40 (GPIO28_ADC2)
- net GPIO28_ADC2: now also J3.4 (Pin_4)
- net GPIO29_ADC3: now reaches U1.41 (GPIO29_ADC3)
- net GPIO29_ADC3: now also J3.2 (Pin_2)
- net at U1.46 (USB_DM): now also R5.2
- net at U1.47 (USB_DP): now also R4.2
- net GPIO3: now reaches U1.5 (GPIO3)
- net GPIO3: now also J2.5 (Pin_5)
- net QSPI_SD3: now reaches U1.51 (QSPI_SD3)
- net QSPI_SD3: now also U3.7 (~{HOLD}/~{RESET}/IO_{3})
- net QSPI_SCLK: now reaches U1.52 (QSPI_SCLK)
- net QSPI_SCLK: now also U3.6 (CLK)
- net QSPI_SD0: now reaches U1.53 (QSPI_SD0)
- net QSPI_SD0: now also U3.5 (DI/IO_{0})
- net QSPI_SD2: now reaches U1.54 (QSPI_SD2)
- net QSPI_SD2: now also U3.3 (~{WP}/IO_{2})
- net QSPI_SD1: now reaches U1.55 (QSPI_SD1)
- net QSPI_SD1: now also U3.2 (DO/IO_{1})
- net QSPI_SS: now reaches U1.56 (QSPI_SS)
- net QSPI_SS: now also R6.2, R7.1, U3.1 (~{CS})
- net GPIO4: now reaches U1.6 (GPIO4)
- net GPIO4: now also J2.6 (Pin_6)
- net GPIO5: now reaches U1.7 (GPIO5)
- net GPIO5: now also J2.7 (Pin_7)
- net GPIO6: now reaches U1.8 (GPIO6)
- net GPIO6: now also J2.9 (Pin_9)
- net GPIO7: now reaches U1.9 (GPIO7)
- net GPIO7: now also J2.10 (Pin_10)
- new net: J1.B5 (CC2), R2.1
- new net: R7.2, SW1.2
- new net: C5.2, SW1.1
- new net: C4.2, R3.1, Y1.1
- new net: J1.A5 (CC1), R1.1
- new net D+: J1.A6 (D+), J1.B6 (D+), R4.1
- new net D-: J1.A7 (D-), J1.B7 (D-), R5.1
- new net VBUS: C1.1, J1.A4 (VBUS), J1.A9 (VBUS), J1.B4 (VBUS), J1.B9 (VBUS), J3.1 (Pin_1), U2.3 (VI)
Other:
- note added: "Crystal Oscillator"
- note added: "Flash Memory IC"
- note added: "RP2040 MCU"
- note added: "USB Receptacle"
- note added: "Voltage Regulator"
- moved on the sheet: U1

Commit message: Add files via upload
Parts:
- added C10, C11, C12, C13, C14, C16, C17, C18, C7, C8, C9: 0.1u, symbol Device:C
- added C15, C6: 1u, symbol Device:C
- C3, C4: value 15p -> C
- R4, R5: value R -> 27
- Y1: value Crystal_GND24 -> 12MHz
Connections:
- net +1V1: now also C15.1, C16.1, C17.1
- net +3V3: now also J3.5 (Pin_5), C10.1, C11.1, C12.1, C13.1, C14.1, C18.2, C6.1, C7.1, C8.1, C9.1
- net GND: now also J2.13 (Pin_13), J2.18 (Pin_18), J2.3 (Pin_3), J2.8 (Pin_8), J3.13 (Pin_13), J3.18 (Pin_18), J3.3 (Pin_3), J3.8 (Pin_8), J4.2 (Pin_2), C10.2, C11.2, C12.2, C13.2, C14.2, C15.2, C16.2, C17.2, C18.1, C6.2, C7.2, C8.2, C9.2
- net GPIO16: now also J3.20 (Pin_20)
- net GPIO17: now also J3.19 (Pin_19)
- net GPIO18: now also J3.17 (Pin_17)
- net GPIO19: now also J3.16 (Pin_16)
- net GPIO20: now also J3.15 (Pin_15)
- net GPIO21: now also J3.14 (Pin_14)
- net GPIO22: now also J3.12 (Pin_12)
- net GPIO26_ADC0: now also J3.7 (Pin_7); no longer J3.5 (Pin_5)
- net GPIO27_ADC1: now also J3.6 (Pin_6)
- net SWCLK: now also J4.1 (Pin_1)
- net SWD: now also J4.3 (Pin_3)
- net RUN: now reaches J3.11 (Pin_11)
Other:
- note added: "Decoupling"
- note added: "Header Pins"
- moved on the sheet: C1, C2, C3, C4, C5, J1, J2, J3, J4, R1, R2, R3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
