File: CTR-0-main/CTR-0-main/CTR-0/CTR-0.kicad_pcb (KiCad board)
At the start: 2 copper layers, 21 x 51 mm, 35 parts, among them J1 USB_C_Receptacle_USB2.0_14P, J2 Conn_01x20, J3 Conn_01x20, J4 Conn_01x03, SW1 SW_Push, U1 RP2040, U2 NCP1117-3.3_SOT223, U3 W25Q128JVS, U4 TVS1400DRV, Y1 12MHz

Commit message: Add files via upload
Parts:
- moved C3 0.25 mm to (189.3, 93.2)
Routing:
- net /SWD: track 0.00 -> 29.7 mm
- net +5V: track 20.4 -> 29.3 mm
- net +3V3: track 40.7 -> 45.5 mm, vias 4 -> 5
- added copper zone on F.Cu, net GND
