File: CTR-0-main/CTR-0-main/CTR-0/CTR-0.kicad_sch (KiCad schematic)
At the start: 35 parts, among them J1 USB_C_Receptacle_USB2.0_14P, J2 Conn_01x20, J3 Conn_01x20, J4 Conn_01x03, SW1 SW_Push, U1 RP2040, U2 NCP1117-3.3_SOT223, U3 W25Q128JVS, U4 TVS1400DRV, Y1 12MHz

Commit message: Add files via upload
Other:
- moved on the sheet: C18
Changed lines of the file:
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@@
 	(wire
 		(pts
+			(xy 109.22 43.18) (xy 107.95 43.18)
+		)
+		(stroke
+			(width 0)
+			(type default)
+		)
+	)
+	(wire
+		(pts
 			(xy 102.87 99.06) (xy 109.22 99.06)
 		)
@@
 	(wire
 		(pts
-			(xy 115.57 43.18) (xy 120.65 43.18)
+			(xy 116.84 43.18) (xy 120.65 43.18)
 		)
 		(stroke
@@
 	(symbol
 		(lib_id "Device:C")
-		(at 111.76 43.18 270)
+		(at 113.03 43.18 270)
 		(unit 1)
 		(exclude_from_sim no)
@@
 		(dnp no)
 		(property "Reference" "C18"
-			(at 114.808 41.91 90)
+			(at 116.078 41.91 90)
 			(effects
 				(font
@@
 		)
 		(property "Value" "100n"
-			(at 115.316 44.45 90)
+			(at 116.586 44.45 90)
 			(effects
 				(font
@@
 		)
 		(property "Footprint" "Capacitor_SMD:C_0402_1005Metric"
-			(at 107.95 44.1452 0)
+			(at 109.22 44.1452 0)
 			(effects
 				(font
@@
 		)
 		(property "Datasheet" "~"
-			(at 111.76 43.18 0)
+			(at 113.03 43.18 0)
 			(effects
 				(font
@@
 		)
 		(property "Description" "Unpolarized capacitor"
-			(at 111.76 43.18 0)
+			(at 113.03 43.18 0)
 			(effects
 				(font
